File: PIC_ESP32.kicad_pcb (KiCad board)
At the start: 2 copper layers, 54 parts, among them J1 USB_B_Micro, J2 12V_SMPS, J3 12V_BATT, J4 BME, J5 LCD, J6 FANS, J7 IR sensor, SW1 EN, SW2 SW_Reed, SW3 FLASH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

Commit message: change 1
Routing:
- net GND: track 1.67 -> 38.1 mm

Commit message: Update PIC_ESP32.kicad_pcb
Routing:
- net Net-(D3-Pad2): track 1.76 -> 23.5 mm
Changed lines of the file:
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@@
     (thickness 1.6)
     (drawings 0)
-    (tracks 37)
+    (tracks 39)
     (zones 0)
     (modules 54)
@@
   (segment (start 92.51188 95.8125) (end 92.51188 97.53282) (width 0.5) (layer F.Cu) (net 5))
   (segment (start 176.0601 97.5623) (end 177.3047 98.8069) (width 2) (layer F.Cu) (net 11))
+  (segment (start 178.308 84.582) (end 171.704 77.978) (width 0.25) (layer F.Cu) (net 11))
+  (segment (start 178.308 96.94) (end 178.308 84.582) (width 0.25) (layer F.Cu) (net 11))
   (segment (start 115.13518 66.36678) (end 115.0497 66.2813) (width 0.25) (layer F.Cu) (net 18))
   (segment (start 103.75646 70.91058) (end 104.82466 69.84238) (width 0.25) (layer F.Cu) (net 20))
